File: PCB/Projet_Final_GI_Equipe2.kicad_pcb (KiCad board)
At the start: 2 copper layers, 100 x 100 mm, 31 parts, among them J1 Conn_01x15_Female, J2 Conn_01x15_Female, J3 mcp2gauche, J4 mcp1gauche, J5 mcp1droite, J6 mcp2droite, SW1 SW_Push, SW2 SW_Push, U1 COM-09032, U2 COM-09032

Commit message: bozoAdd
Parts:
- moved D3 126.4 mm to (235.8, 86.0)
- moved D2 116.6 mm to (225.2, 86.5)
- moved D1 108.1 mm to (215.5, 86.2)
- moved D5 102.6 mm to (218.2, 104.8)
- moved D4 67.3 mm to (246.2, 86.2)
- moved D8 58.3 mm to (244.0, 105.0)
- moved D7 56.0 mm to (235.5, 105.0)
- moved D6 41.4 mm to (227.2, 104.8)
Other:
- board size 100 x 100 mm -> 104.8 x 99.1 mm
Changed lines of the file:
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@@
   (net 42 "/R3")
   (footprint "LED_SMD:LED_WS2812B_PLCC4_5.0x5.0mm_P3.2mm" (layer "F.Cu")
-    (at 181 118)
+    (at 235.5 105)
     (descr "https://cdn-shop.adafruit.com/datasheets/WS2812B.pdf")
     (tags "LED RGB NeoPixel")
@@
   )
   (footprint "LED_SMD:LED_WS2812B_PLCC4_5.0x5.0mm_P3.2mm" (layer "F.Cu")
-    (at 179 88)
+    (at 246.25 86.25)
     (descr "https://cdn-shop.adafruit.com/datasheets/WS2812B.pdf")
     (tags "LED RGB NeoPixel")
@@
   )
   (footprint "LED_SMD:LED_WS2812B_PLCC4_5.0x5.0mm_P3.2mm" (layer "F.Cu")
-    (at 117 88)
+    (at 218.25 104.75)
     (descr "https://cdn-shop.adafruit.com/datasheets/WS2812B.pdf")
     (tags "LED RGB NeoPixel")
@@
   )
   (footprint "LED_SMD:LED_WS2812B_PLCC4_5.0x5.0mm_P3.2mm" (layer "F.Cu")
-    (at 186 99)
+    (at 244 105)
     (descr "https://cdn-shop.adafruit.com/datasheets/WS2812B.pdf")
     (tags "LED RGB NeoPixel")
@@
   )
   (footprint "LED_SMD:LED_WS2812B_PLCC4_5.0x5.0mm_P3.2mm" (layer "F.Cu")
-    (at 113 116)
+    (at 235.75 86)
     (descr "https://cdn-shop.adafruit.com/datasheets/WS2812B.pdf")
     (tags "LED RGB NeoPixel")
@@
   )
   (footprint "LED_SMD:LED_WS2812B_PLCC4_5.0x5.0mm_P3.2mm" (layer "F.Cu")
-    (at 109 96)
+    (at 225.25 86.5)
     (descr "https://cdn-shop.adafruit.com/datasheets/WS2812B.pdf")
     (tags "LED RGB NeoPixel")
@@
   )
   (footprint "LED_SMD:LED_WS2812B_PLCC4_5.0x5.0mm_P3.2mm" (layer "F.Cu")
-    (at 186 108)
+    (at 227.25 104.75)
     (descr "https://cdn-shop.adafruit.com/datasheets/WS2812B.pdf")
     (tags "LED RGB NeoPixel")
@@
   )
   (footprint "LED_SMD:LED_WS2812B_PLCC4_5.0x5.0mm_P3.2mm" (layer "F.Cu")
-    (at 109 105)
+    (at 215.5 86.25)
     (descr "https://cdn-shop.adafruit.com/datasheets/WS2812B.pdf")
     (tags "LED RGB NeoPixel")
@@
     )
   )
-  (gr_rect (start 98 53) (end 198 153) (layer "Edge.Cuts") (width 0.1) (fill none))
-  (gr_poly
-    (pts
-      (xy 197 152)
-      (xy 176 152)
-      (xy 176 121)
-      (xy 118 121)
-      (xy 118 152)
-      (xy 98 152)
-      (xy 98 53)
-      (xy 197 53)
-    ) (layer "Edge.Cuts") (width 0.1) (fill none))
+  (gr_line (start 175.75 152) (end 176.5 152) (layer "Edge.Cuts") (width 0.1))
+  (gr_line (start 200.244796 147.744796) (end 200.5 58.389087) (layer "Edge.Cuts") (width 0.1))
+  (gr_line (start 195 52.889087) (end 101.25 53) (layer "Edge.Cuts") (width 0.1))
+  (gr_line (start 95.75 147.75) (end 95.75 58.5) (layer "Edge.Cuts") (width 0.1))
+  (gr_arc (start 200.244796 147.744796) (mid 199 150.75) (end 195.994796 151.994796) (layer "Edge.Cuts") (width 0.1))
+  (gr_line (start 176.5 152) (end 175.75 152) (layer "Edge.Cuts") (width 0.1))
+  (gr_line (start 120.75 152) (end 118.75 152) (layer "Edge.Cuts") (width 0.1))
+  (gr_line (start 100 152) (end 118.75 152) (layer "Edge.Cuts") (width 0.1))
+  (gr_arc (start 168.75 121.5) (mid 171.755204 122.744796) (end 173 125.75) (layer "Edge.Cuts") (width 0.1))
+  (gr_line (start 122.505204 125.755204) (end 120.75 152) (layer "Edge.Cuts") (width 0.1))
+  (gr_line (start 126.755204 121.505204) (end 168.75 121.5) (layer "Edge.Cuts") (width 0.1))
+  (gr_arc (start 95.75 58.5) (mid 97.360913 54.610913) (end 101.25 53) (layer "Edge.Cuts") (width 0.1))
+  (gr_arc (start 122.505204 125.755204) (mid 123.75 122.75) (end 126.755204 121.505204) (layer "Edge.Cuts") (width 0.1))
+  (gr_line (start 195.994796 151.994796) (end 176.5 152) (layer "Edge.Cuts") (width 0.1))
+  (gr_arc (start 100 152) (mid 96.994796 150.755204) (end 95.75 147.75) (layer "Edge.Cuts") (width 0.1))
+  (gr_arc (start 195 52.889087) (mid 198.889087 54.5) (end 200.5 58.389087) (layer "Edge.Cuts") (width 0.1))
+  (gr_line (start 173 125.75) (end 175.75 152) (layer "Edge.Cuts") (width 0.1))
+  (gr_line (start 118.75 152) (end 120.75 152) (layer "Edge.Cuts") (width 0.1))
 )
