File: PCB/Projet_Final_GI_Equipe2.kicad_pcb (KiCad board)
At the start: 2 copper layers, 104.8 x 99.1 mm, 31 parts, among them J1 Conn_01x15_Female, J2 Conn_01x15_Female, J3 mcp2gauche, J4 mcp1gauche, J5 mcp1droite, J6 mcp2droite, SW1 SW_Push, SW2 SW_Push, U1 COM-09032, U2 COM-09032

Commit message: DEBIANROUILLE TOI
Parts:
- removed C2, C4, C6, C8: 0.1 uF, Capacitor_SMD:C_0805_2012Metric_Pad1.18x1.45mm_HandSolder
- removed D2, D4, D6, D8: WS2812B, LED_SMD:LED_WS2812B_PLCC4_5.0x5.0mm_P3.2mm
- SW1, SW2: footprint Button_Switch_THT:KSA_Tactile_SPST -> Button_Switch_THT:SW_PUSH-12mm
- moved D3 134.6 mm to (103.9, 59.2), turned to -90 degrees
- moved D1 112.9 mm to (103.9, 69.2), turned to -90 degrees
- moved C5 81.6 mm to (186.2, 59.9), turned to -90 degrees
- moved SW2 79.9 mm to (184.7, 85.3)
- moved C3 78.1 mm to (98.0, 59.7), turned to 90 degrees
- moved C1 72.4 mm to (98.0, 69.1), turned to 90 degrees
- moved R1 68.4 mm to (113.8, 68.3), turned to 180 degrees
- moved C7 68.3 mm to (186.4, 69.1), turned to -90 degrees
- moved R6 62.4 mm to (123.4, 85.1)
- moved R3 60.3 mm to (196.1, 97.3), turned to 180 degrees
- moved R2 59.9 mm to (99.8, 97.3)
- moved D7 56.4 mm to (191.9, 69.2), turned to 90 degrees
- moved J4 55.1 mm to (116.2, 77.5)
- moved J5 54.4 mm to (116.2, 62.2)
- moved D5 52.6 mm to (191.9, 59.2), turned to 90 degrees
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Connections:
- D7 pad 2: Net-(D2-Pad4) -> unconnected-(D7-Pad2)
- J1 pad 4: /S3 -> /S3/R3
- J1 pad 5: /S2 -> /S2/L3
- R6 pad 2: /L3 -> /S2/L3
- R7 pad 2: /R3 -> /S3/R3
- U1 pad B1A: /L3 -> /S2/L3
- U2 pad B1A: /R3 -> /S3/R3
Routing:
- net GND: track 0.00 -> 311.6 mm
- net /3V3: track 0.00 -> 241.9 mm
- net /5V: track 0.00 -> 159.1 mm
- net /3.3V: track 0.00 -> 137.3 mm
- net /G: track 0.00 -> 104.7 mm
- net Net-(D3-Pad2): track 0.00 -> 90.4 mm
- net /D6/DOUT: track 0.00 -> 86.0 mm
- net /D7/DIN: track 0.00 -> 85.4 mm
- net /D2/SPECIAL: track 0.00 -> 83.5 mm
- net /D1/ATTACK: track 0.00 -> 62.1 mm
- net /D5/CLK: track 0.00 -> 59.1 mm
- net /D4/CSL: track 0.00 -> 47.7 mm
- net /D8/CSR: track 0.00 -> 46.5 mm
- net /LEFTH: track 0.00 -> 42.8 mm
- net /RIGHTH: track 0.00 -> 39.7 mm
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
Commit message: tu peux envoyer tes points, Jessy
Parts:
- added C2: 10uF, Capacitor_SMD:C_0805_2012Metric_Pad1.18x1.45mm_HandSolder, B.Cu at (153.4, 107.7)
- added C4: 22uF, Capacitor_SMD:C_0805_2012Metric_Pad1.18x1.45mm_HandSolder, B.Cu at (153.4, 103.1)
- added J7: Conn_01x03_Male, Connector_PinHeader_2.54mm:PinHeader_1x03_P2.54mm_Vertical, F.Cu at (144.0, 94.0)
- added J8: Conn_01x02_Male, Connector_PinHeader_2.54mm:PinHeader_1x02_P2.54mm_Vertical, F.Cu at (146.0, 119.4)
- added JP1: SolderJumper_2_Open, Jumper:SolderJumper-2_P1.3mm_Open_RoundedPad1.0x1.5mm, F.Cu at (126.0, 82.3)
- added JP2: SolderJumper_2_Open, Jumper:SolderJumper-2_P1.3mm_Open_RoundedPad1.0x1.5mm, F.Cu at (170.9, 82.3)
- added U3: AZ1117-5.0, Package_TO_SOT_SMD:SOT-223, B.Cu at (146.8, 104.4)
- moved R7 2.34 mm to (170.9, 85.3)
Connections:
- R6 pad 2: /S2/L3 -> Net-(R6-Pad2)
- R7 pad 2: /S3/R3 -> Net-(R7-Pad2)
- U1 pad B1A: /S2/L3 -> Net-(R6-Pad2)
- U2 pad B1A: /S3/R3 -> Net-(R7-Pad2)
Routing:
- net /G: track 104.7 -> 144.3 mm
- net /PLUS: track 0.00 -> 32.1 mm
- net /VIN: track 0.00 -> 22.9 mm, vias 0 -> 1
- net Net-(C4-Pad2): track 0.00 -> 15.4 mm
- net GND: track 311.6 -> 326.0 mm
- net Net-(R7-Pad2): track 0.00 -> 12.9 mm
- net /S2/L3: track 25.5 -> 15.0 mm
- net Net-(R6-Pad2): track 0.00 -> 10.3 mm
- net /3V3: track 241.9 -> 246.7 mm
- net /S3/R3: track 37.6 -> 35.2 mm, vias 0 -> 1
- added copper zone on B.Cu, net /G
- added copper zone on F.Cu, net /G
Other:
- board text added: "- +"
- board text added: "BAT REG"
- board text added: "Marc-Étienne Gendron-Fontaine Jessy Grimard-Maheux Zachary Poulin Mohammad Barin Wahidi TGE - TSO - GI Cégep de Sherbrooke 2022/11/16"
- board text added: "▲"

Commit message: PCB fix
Connections:
- C1 pad 2: /5V -> /3.3V
- C3 pad 2: /5V -> /3.3V
- C5 pad 2: /5V -> /3.3V
- C7 pad 2: /5V -> /3.3V
- D1 pad 1: /5V -> /3.3V
- D3 pad 1: /5V -> /3.3V
- D5 pad 1: /5V -> /3.3V
- D7 pad 1: /5V -> /3.3V
- J1 pad 10: /G -> GND
- J1 pad 11: /3V3 -> /3.3V
- J1 pad 14: /G -> GND
- J1 pad 2: /G -> GND
- J2 pad 14: /G -> GND
- J2 pad 15: /3V3 -> /3.3V
- J2 pad 6: /3V3 -> /3.3V
- J2 pad 7: /G -> GND
- J8 pad 1: /G -> GND
- R6 pad 1: /3V3 -> /3.3V
- R7 pad 1: /3V3 -> /3.3V
- U1 pad H1: /3V3 -> /3.3V
- U1 pad V1: /3V3 -> /3.3V
- U2 pad H1: /3V3 -> /3.3V
- U2 pad V1: /3V3 -> /3.3V
Routing:
- net /3.3V: track 137.3 -> 550.9 mm, vias 0 -> 1
- net /3V3: track 246.7 -> 0.00 mm
- net /5V: track 159.1 -> 0.00 mm
- net GND: track 326.0 -> 470.3 mm
- net /G: track 144.3 -> 0.00 mm
- added copper zone on B.Cu, net GND
- added copper zone on F.Cu, net GND
- removed copper zone on B.Cu, net /G
- removed copper zone on F.Cu, net /G

Commit message: Version final PCB Zachary
Parts:
- moved J3 6.85 mm to (178.0, 77.5)
- moved J6 6.85 mm to (178.0, 62.2)
- moved J5 6.15 mm to (110.0, 62.0)
- moved J4 6.15 mm to (110.0, 77.2)
- moved R1 5.83 mm to (108.0, 69.0)
- moved C5 3.82 mm to (190.0, 60.0)
- moved C7 3.56 mm to (190.0, 69.1)
- moved D5 3.11 mm to (195.0, 59.2)
- moved D7 3.11 mm to (195.0, 69.2)
- moved D1 2.89 mm to (101.0, 69.2)
- moved D3 2.89 mm to (101.0, 59.2)
- moved C3 2.07 mm to (96.0, 60.0)
- moved C1 2.04 mm to (96.0, 69.1)
- moved R2 1.72 mm to (99.8, 99.0)
- moved R3 1.72 mm to (196.1, 99.0)
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Routing:
- net /3.3V: track 550.9 -> 595.9 mm
- net GND: track 470.3 -> 498.9 mm, vias 0 -> 1
- net /D7/DIN: track 85.4 -> 105.5 mm
- net /D6/DOUT: track 86.0 -> 105.7 mm
- net /D5/CLK: track 59.1 -> 72.9 mm
- net /D8/CSR: track 46.5 -> 55.4 mm
- net /D0/RGB: track 24.6 -> 33.3 mm
- net /D4/CSL: track 47.7 -> 54.0 mm
- net Net-(D3-Pad2): track 90.3 -> 96.0 mm
- net /RIGHTH: track 39.7 -> 42.5 mm
- net /RIGHTV: track 34.1 -> 36.9 mm
- net /LEFTV: track 29.6 -> 31.7 mm
- net Net-(D1-Pad4): track 8.64 -> 6.62 mm
- net /D1/ATTACK: track 62.1 -> 63.1 mm
- net /D2/SPECIAL: track 83.5 -> 84.2 mm
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Other:
- board size 104.8 x 99.1 mm -> 111 x 99.1 mm
