File: PCB/Projet_Final_GI_Equipe2.kicad_sch (KiCad schematic)
At the start: 6 parts, among them SW1 SW_Push, SW2 SW_Push, SW3 SW_Push, SW4 SW_Push, U1 COM-09032, U2 COM-09032

Commit message: Modif PCB
Parts:
- removed SW2, SW3, SW4: SW_Push, symbol Switch:SW_Push
- added C? (x8): 0.1 uF, symbol Device:C
- added D? (x8): WS2812B, LED_SMD:LED_WS2812B_PLCC4_5.0x5.0mm_P3.2mm, symbol LED:WS2812B
- added J? (x2): Conn_01x15_Female, symbol Connector:Conn_01x15_Female
- added R? (x6): 1K, symbol Device:R_US
- added SW? (x3): SW_Push, symbol Switch:SW_Push
Connections:
- net 3.3V: now also SW?.1, SW?.1, SW?.1
- net L3: now reaches U1.B1A (SEL+)
- net L3: now also R?.2
- net GND: now reaches U1.B2A (SEL-)
- net GND: now also U1.H3 (H-), U1.S1 (SHIELD), U1.S2 (SHIELD), U1.S3 (SHIELD), U1.S4 (SHIELD), U1.V3 (V-), U2.B2A (SEL-), U2.H3 (H-), U2.S1 (SHIELD), U2.S2 (SHIELD), U2.S3 (SHIELD), U2.S4 (SHIELD), U2.V3 (V-), C?.1, C?.1, C?.1, C?.1, C?.1, C?.1, C?.1, C?.1, D?.3 (VSS), D?.3 (VSS), D?.3 (VSS), D?.3 (VSS), D?.3 (VSS), D?.3 (VSS), D?.3 (VSS), D?.3 (VSS), R?.2, R?.2, R?.2, R?.2
- net 3V3: now reaches U1.H1 (H+)
- net 3V3: now also U1.V1 (V+), U2.H1 (H+), U2.V1 (V+), J?.11 (Pin_11), J?.15 (Pin_15), J?.6 (Pin_6), R?.1, R?.1
- net LEFTH: now reaches U1.H2 (H)
- net LEFTV: now reaches U1.V2 (V)
- net R3: now reaches U2.B1A (SEL+)
- net R3: now also R?.2
- net RIGHTH: now reaches U2.H2 (H)
- net RIGHTV: now reaches U2.V2 (V)
- net UP: now reaches SW1.2
- net UP: now also R?.1
- new net: D?.2 (DOUT), D?.4 (DIN) (x6)
- new net 5V: C?.2, C?.2, C?.2, C?.2, C?.2, C?.2, C?.2, C?.2, D?.1 (VDD), D?.1 (VDD), D?.1 (VDD), D?.1 (VDD), D?.1 (VDD), D?.1 (VDD), D?.1 (VDD), D?.1 (VDD)
- new net A0: J?.1 (Pin_1)
- new net D0: J?.1 (Pin_1)
- new net D1: J?.2 (Pin_2)
- new net D2: J?.3 (Pin_3)
- new net D3: J?.4 (Pin_4)
- new net D4: J?.5 (Pin_5)
- new net D5: J?.8 (Pin_8)
- new net D6: J?.9 (Pin_9)
- new net D7: J?.10 (Pin_10)
- new net D8: J?.11 (Pin_11)
- new net DOWN: R?.1, SW?.2
- new net EN: J?.12 (Pin_12)
- new net G: J?.10 (Pin_10), J?.14 (Pin_14), J?.14 (Pin_14), J?.2 (Pin_2), J?.7 (Pin_7)
- new net LEFT: R?.1, SW?.2
- new net LEFT_RGB: D?.4 (DIN)
- new net RIGHT: R?.1, SW?.2
- new net RIGHT_RGB: D?.4 (DIN)
- new net RST: J?.13 (Pin_13)
- new net RX: J?.12 (Pin_12)
- new net S1: J?.6 (Pin_6)
- new net S2: J?.5 (Pin_5)
- new net S3: J?.4 (Pin_4)
- new net SC: J?.7 (Pin_7)
- new net SK: J?.9 (Pin_9)
- new net SO: J?.8 (Pin_8)
- new net TX: J?.13 (Pin_13)
- new net VIN: J?.15 (Pin_15)
- new net VV: J?.3 (Pin_3)
Other:
- moved on the sheet: SW1

Commit message: Schema 2.0
Parts:
- added U? (x2): MCP3202, symbol Analog_ADC:MCP3202
Connections:
- net 3.3V: now also U?.8 (VDD/VREF), U?.8 (VDD/VREF)
- net GND: now also U?.4 (VSS), U?.4 (VSS)
- net LEFTH: now also U?.3 (CH1)
- net LEFTV: now also U?.2 (CH0)
- net RIGHTH: now also U?.3 (CH1)
- net RIGHTV: now also U?.2 (CH0)
- new net: U?.5 (DIN), U?.5 (DIN)
- new net: U?.6 (DOUT), U?.6 (DOUT)
- new net: U?.7 (CLK), U?.7 (CLK)
Changed lines of the file:
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@@
+    (stroke (width 0) (type default) (color 0 0 0 0))
+  )
+  (wire (pts (xy 259.588 131.826) (xy 259.588 97.536))
     (stroke (width 0) (type default) (color 0 0 0 0))
   )
@@
     (stroke (width 0) (type default) (color 0 0 0 0))
   )
+  (wire (pts (xy 235.966 141.986) (xy 235.966 143.256))
+    (stroke (width 0) (type default) (color 0 0 0 0))
+  )
   (wire (pts (xy 163.83 94.742) (xy 167.386 94.742))
     (stroke (width 0) (type default) (color 0 0 0 0))
@@
     (stroke (width 0) (type default) (color 0 0 0 0))
   )
+  (wire (pts (xy 252.73 100.076) (xy 257.048 100.076))
+    (stroke (width 0) (type default) (color 0 0 0 0))
+  )
+  (wire (pts (xy 253.746 131.826) (xy 259.588 131.826))
+    (stroke (width 0) (type default) (color 0 0 0 0))
+  )
   (wire (pts (xy 163.576 104.902) (xy 167.386 104.902))
     (stroke (width 0) (type default) (color 0 0 0 0))
@@
     (stroke (width 0) (type default) (color 0 0 0 0))
   )
+  (wire (pts (xy 259.588 97.536) (xy 252.73 97.536))
+    (stroke (width 0) (type default) (color 0 0 0 0))
+  )
   (wire (pts (xy 25.146 130.048) (xy 25.146 132.334))
     (stroke (width 0) (type default) (color 0 0 0 0))
@@
     (stroke (width 0) (type default) (color 0 0 0 0))
   )
+  (wire (pts (xy 253.746 134.366) (xy 257.048 134.366))
+    (stroke (width 0) (type default) (color 0 0 0 0))
+  )
   (wire (pts (xy 50.546 166.624) (xy 62.738 166.624))
     (stroke (width 0) (type default) (color 0 0 0 0))
@@
     (stroke (width 0) (type default) (color 0 0 0 0))
   )
+  (wire (pts (xy 234.95 107.696) (xy 234.95 108.458))
+    (stroke (width 0) (type default) (color 0 0 0 0))
+  )
+  (wire (pts (xy 257.048 100.076) (xy 257.048 134.366))
+    (stroke (width 0) (type default) (color 0 0 0 0))
+  )
   (wire (pts (xy 50.546 130.048) (xy 50.546 132.334))
     (stroke (width 0) (type default) (color 0 0 0 0))
@@
     (stroke (width 0) (type default) (color 0 0 0 0))
   )
+  (wire (pts (xy 262.128 92.456) (xy 252.73 92.456))
+    (stroke (width 0) (type default) (color 0 0 0 0))
+  )
   (wire (pts (xy 72.898 84.836) (xy 72.898 75.946))
     (stroke (width 0) (type default) (color 0 0 0 0))
@@
     (stroke (width 0) (type default) (color 0 0 0 0))
   )
+  (wire (pts (xy 253.746 126.746) (xy 262.128 126.746))
+    (stroke (width 0) (type default) (color 0 0 0 0))
+  )
   (wire (pts (xy 119.888 109.982) (xy 119.888 113.03))
     (stroke (width 0) (type default) (color 0 0 0 0))
@@
     (stroke (width 0) (type default) (color 0 0 0 0))
   )
+  (wire (pts (xy 262.128 126.746) (xy 262.128 92.456))
+    (stroke (width 0) (type default) (color 0 0 0 0))
+  )
   (wire (pts (xy 73.152 100.076) (xy 73.152 91.186))
     (stroke (width 0) (type default) (color 0 0 0 0))
@@
     (effects (font (size 1.27 1.27)) (justify right bottom))
   )
+  (label "3.3V" (at 235.966 116.586 180)
+    (effects (font (size 1.27 1.27)) (justify right bottom))
+  )
   (label "G" (at 182.372 41.402 180)
     (effects (font (size 1.27 1.27)) (justify right bottom))
@@
     (effects (font (size 1.27 1.27)) (justify right bottom))
   )
+  (label "RIGHTV" (at 223.266 124.206 180)
+    (effects (font (size 1.27 1.27)) (justify right bottom))
+  )
   (label "D3" (at 203.2 46.482 0)
     (effects (font (size 1.27 1.27)) (justify left bottom))
@@
     (effects (font (size 1.27 1.27)) (justify left bottom))
   )
+  (label "3.3V" (at 234.95 82.296 180)
+    (effects (font (size 1.27 1.27)) (justify right bottom))
+  )
   (label "5V" (at 25.146 130.048 0)
     (effects (font (size 1.27 1.27)) (justify left bottom))
@@
     (effects (font (size 1.27 1.27)) (justify right bottom))
   )
+  (label "LEFTV" (at 222.25 89.916 180)
+    (effects (font (size 1.27 1.27)) (justify right bottom))
+  )
   (label "3V3" (at 112.268 109.982 180)
     (effects (font (size 1.27 1.27)) (justify right bottom))
@@
     (effects (font (size 1.27 1.27)) (justify right bottom))
   )
+  (label "LEFTH" (at 222.25 100.076 180)
+    (effects (font (size 1.27 1.27)) (justify right bottom))
+  )
   (label "D5" (at 203.2 56.642 0)
     (effects (font (size 1.27 1.27)) (justify left bottom))
+  )
+  (label "RIGHTH" (at 223.266 134.366 180)
+    (effects (font (size 1.27 1.27)) (justify right bottom))
   )
   (label "TX" (at 203.2 69.342 0)
@@
     (pin "2")
   )
+  (symbol (lib_id "Analog_ADC:MCP3202") (at 235.966 129.286 0) (unit 1)
+    (in_bom yes) (on_board yes) (fields_autoplaced)
+    (property "Reference" "U?" (id 0) (at 237.9854 114.3 0)
+      (effects (font (size 1.27 1.27)) (justify left))
+    )
+    (property "Value" "MCP3202" (id 1) (at 237.9854 116.84 0)
+      (effects (font (size 1.27 1.27)) (justify left))
+    )
+    (property "Footprint" "" (id 2) (at 235.966 131.826 0)
+      (effects (font (size 1.27 1.27)) hide)
+    )
+    (property "Datasheet" "http://ww1.microchip.com/downloads/en/DeviceDoc/21034D.pdf" (id 3) (at 235.966 124.206 0)
+      (effects (font (size 1.27 1.27)) hide)
+    )
+    (pin "1")
+    (pin "2")
+    (pin "3")
+    (pin "4")
+    (pin "5")
+    (pin "6")
+    (pin "7")
+    (pin "8")
+  )
   (symbol (lib_id "power:GND") (at 80.01 54.102 0) (unit 1)
     (in_bom yes) (on_board yes) (fields_autoplaced)
@@
     )
     (property "Datasheet" "" (id 3) (at 80.01 54.102 0)
+      (effects (font (size 1.27 1.27)) hide)
+    )
+    (pin "1")
+  )
+  (symbol (lib_id "power:GND") (at 235.966 143.256 0) (unit 1)
+    (in_bom yes) (on_board yes) (fields_autoplaced)
+    (property "Reference" "#PWR?" (id 0) (at 235.966 149.606 0)
+      (effects (font (size 1.27 1.27)) hide)
+    )
+    (property "Value" "GND" (id 1) (at 235.966 148.59 0))
+    (property "Footprint" "" (id 2) (at 235.966 143.256 0)
+      (effects (font (size 1.27 1.27)) hide)
+    )
+    (property "Datasheet" "" (id 3) (at 235.966 143.256 0)
       (effects (font (size 1.27 1.27)) hide)
     )
@@
     (pin "1")
     (pin "2")
+  )
+  (symbol (lib_id "power:GND") (at 234.95 108.458 0) (unit 1)
+    (in_bom yes) (on_board yes) (fields_autoplaced)
+    (property "Reference" "#PWR?" (id 0) (at 234.95 114.808 0)
+      (effects (font (size 1.27 1.27)) hide)
+    )
+    (property "Value" "GND" (id 1) (at 234.95 113.03 0))
+    (property "Footprint" "" (id 2) (at 234.95 108.458 0)
+      (effects (font (size 1.27 1.27)) hide)
+    )
+    (property "Datasheet" "" (id 3) (at 234.95 108.458 0)
+      (effects (font (size 1.27 1.27)) hide)
+    )
+    (pin "1")
   )
   (symbol (lib_id "power:GND") (at 113.792 189.484 0) (unit 1)
@@
     (pin "1")
   )
+  (symbol (lib_id "Analog_ADC:MCP3202") (at 234.95 94.996 0) (unit 1)
+    (in_bom yes) (on_board yes) (fields_autoplaced)
+    (property "Reference" "U?" (id 0) (at 236.9694 80.01 0)
+      (effects (font (size 1.27 1.27)) (justify left))
+    )
+    (property "Value" "MCP3202" (id 1) (at 236.9694 82.55 0)
+      (effects (font (size 1.27 1.27)) (justify left))
+    )
+    (property "Footprint" "" (id 2) (at 234.95 97.536 0)
+      (effects (font (size 1.27 1.27)) hide)
+    )
+    (property "Datasheet" "http://ww1.microchip.com/downloads/en/DeviceDoc/21034D.pdf" (id 3) (at 234.95 89.916 0)
+      (effects (font (size 1.27 1.27)) hide)
+    )
+    (pin "1")
+    (pin "2")
+    (pin "3")
+    (pin "4")
+    (pin "5")
+    (pin "6")
+    (pin "7")
+    (pin "8")
+  )
   (symbol (lib_id "power:GND") (at 120.65 104.902 0) (unit 1)
     (in_bom yes) (on_board yes)
@@
       (reference "#PWR?") (unit 1) (value "GND") (footprint "")
     )
+    (path "/3a2c958d-7de0-47a9-a851-0ba12b7f918c"
+      (reference "#PWR?") (unit 1) (value "GND") (footprint "")
+    )
     (path "/4c61f118-0e9e-4e48-a243-d9e267dc4b10"
       (reference "#PWR?") (unit 1) (value "GND") (footprint "")
@@
     )
     (path "/5e3fa9e9-ce73-4f74-b088-3352203b0534"
+      (reference "#PWR?") (unit 1) (value "GND") (footprint "")
+    )
+    (path "/876694f5-ecb0-4846-b2aa-609c9416c1cf"
       (reference "#PWR?") (unit 1) (value "GND") (footprint "")
     )
@@
       (reference "U2") (unit 1) (value "COM-09032") (footprint "XDCR_COM-09032")
     )
-  )
+    (path "/2faae2bb-a0c2-4054-ae9f-2d25525a48e8"
+      (reference "U?") (unit 1) (value "MCP3202") (footprint "")
+    )
+    (path "/c06b07a5-81e8-4fba-b75f-eafa053e1406"
+      (reference "U?") (unit 1) (value "MCP3202") (footprint "")
+    )
+  )

Commit message: Jessy doit finir le PCB
Parts:
- removed R? (x2): 1K, symbol Device:R_US
- removed SW? (x2): SW_Push, symbol Switch:SW_Push
- removed U? (x2): MCP3202, symbol Analog_ADC:MCP3202
- added J3: mcp2gauche, Connector_PinSocket_2.54mm:PinSocket_1x04_P2.54mm_Vertical, symbol Connector:Conn_01x04_Female
- added J4: mcp1gauche, Connector_PinSocket_2.54mm:PinSocket_1x04_P2.54mm_Vertical, symbol Connector:Conn_01x04_Female
- added J5: mcp1droite, Connector_PinSocket_2.54mm:PinSocket_1x04_P2.54mm_Vertical, symbol Connector:Conn_01x04_Female
- added J6: mcp2droite, Connector_PinSocket_2.54mm:PinSocket_1x04_P2.54mm_Vertical, symbol Connector:Conn_01x04_Female
- added R1: 330, Capacitor_SMD:C_0805_2012Metric_Pad1.18x1.45mm_HandSolder, symbol Device:R_US
- C1, C2, C3, C4, C5, C6, C7, C8: renamed from C?; footprint (none) -> Capacitor_SMD:C_0805_2012Metric_Pad1.18x1.45mm_HandSolder
- J1, J2: renamed from J?; footprint (none) -> Connector_PinSocket_2.54mm:PinSocket_1x15_P2.54mm_Vertical
- R2, R3, R6, R7: renamed from R?; footprint (none) -> Capacitor_SMD:C_0805_2012Metric_Pad1.18x1.45mm_HandSolder
- SW1: footprint (none) -> Button_Switch_THT:KSA_Tactile_SPST
- SW2: renamed from SW?; footprint (none) -> Button_Switch_THT:KSA_Tactile_SPST
- U1, U2: footprint XDCR_COM-09032 -> COM-09032:XDCR_COM-09032
- gave numbers to parts that had none: 8
Connections:
- net DOWN is gone; now on net D2/SPECIAL: R3.1, SW2.2
- net RIGHT_RGB is gone; now on an unnamed net: D2.4 (DIN)
- net UP is gone; now on net D1/ATTACK: R2.1, SW1.2
- net 3.3V: now also J5.1 (Pin_1), J6.1 (Pin_1)
- net GND: now also J3.4 (Pin_4), J4.4 (Pin_4)
- net LEFTH: now also J4.3 (Pin_3)
- net LEFTV: now also J4.2 (Pin_2)
- net RIGHTH: now also J3.3 (Pin_3)
- net RIGHTV: now also J3.2 (Pin_2)
- net D0 renamed D0/RGB
- net D0/RGB: now also R1.1
- net D1 renamed D1/ATTACK
- net D2 renamed D2/SPECIAL
- net D4 renamed D4/CSL
- net D4/CSL: now also J4.1 (Pin_1)
- net D5 renamed D5/CLK
- net D5/CLK: now also J5.2 (Pin_2), J6.2 (Pin_2)
- net D6 renamed D6/DOUT
- net D6/DOUT: now also J5.3 (Pin_3), J6.3 (Pin_3)
- net D7 renamed D7/DIN
- net D7/DIN: now also J5.4 (Pin_4), J6.4 (Pin_4)
- net D8 renamed D8/CSR
- net D8/CSR: now also J3.1 (Pin_1)
- net LEFT_RGB: no longer names the net of D1.4 (DIN)
- net LEFT_RGB: now also R1.2
- no-connect marks 0 -> 1
Other:
- company: (none) -> Cégep de Sherbrooke
- title: (none) -> Manette_Robot_NAO
- moved on the sheet: R2, R3, SW1, SW2

Commit message: Jessy doit finir le PCB
Connections:
- net S2 is gone; now on net S2/L3: J1.5 (Pin_5)
- net S3 is gone; now on net S3/R3: J1.4 (Pin_4)
- net L3 renamed S2/L3
- net R3 renamed S3/R3
Changed lines of the file:
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@@
     (effects (font (size 1.27 1.27)) (justify right bottom))
   )
-  (label "S2" (at 182.372 49.022 180)
+  (label "S2{slash}L3" (at 182.372 49.022 180)
     (effects (font (size 1.27 1.27)) (justify right bottom))
   )
@@
     (effects (font (size 1.27 1.27)) (justify right bottom))
   )
-  (label "L3" (at 116.332 113.03 180)
+  (label "S2{slash}L3" (at 116.332 113.03 180)
     (effects (font (size 1.27 1.27)) (justify right bottom))
   )
@@
     (effects (font (size 1.27 1.27)) (justify right bottom))
   )
-  (label "S3" (at 182.372 46.482 180)
+  (label "S3{slash}R3" (at 182.372 46.482 180)
     (effects (font (size 1.27 1.27)) (justify right bottom))
   )
@@
     (effects (font (size 1.27 1.27)) (justify left bottom))
   )
-  (label "R3" (at 159.258 113.03 180)
+  (label "S3{slash}R3" (at 159.258 113.03 180)
     (effects (font (size 1.27 1.27)) (justify right bottom))
   )

Commit message: DEBIANROUILLE TOI
Parts:
- removed C2, C4, C6, C8: 0.1 uF, Capacitor_SMD:C_0805_2012Metric_Pad1.18x1.45mm_HandSolder, symbol Device:C
- removed D2, D4, D6, D8: WS2812B, LED_SMD:LED_WS2812B_PLCC4_5.0x5.0mm_P3.2mm, symbol LED:WS2812B
- SW1, SW2: footprint Button_Switch_THT:KSA_Tactile_SPST -> Button_Switch_THT:SW_PUSH-12mm

Commit message: tu peux envoyer tes points, Jessy
Parts:
- added C2: 10uF, Capacitor_SMD:C_0805_2012Metric_Pad1.18x1.45mm_HandSolder, symbol Device:C
- added C4: 22uF, Capacitor_SMD:C_0805_2012Metric_Pad1.18x1.45mm_HandSolder, symbol Device:C
- added J7: Conn_01x03_Male, Connector_PinHeader_2.54mm:PinHeader_1x03_P2.54mm_Vertical, symbol Connector:Conn_01x03_Male
- added J8: Conn_01x02_Male, Connector_PinHeader_2.54mm:PinHeader_1x02_P2.54mm_Vertical, symbol Connector:Conn_01x02_Male
- added JP1, JP2: SolderJumper_2_Open, Jumper:SolderJumper-2_P1.3mm_Open_RoundedPad1.0x1.5mm, symbol Jumper:SolderJumper_2_Open
- added U3: AZ1117-5.0, Package_TO_SOT_SMD:SOT-223, symbol Regulator_Linear:AZ1117-5.0
Connections:
- net G: now also J8.1 (Pin_1)
- net GND: now also C2.1, C4.1, U3.1 (GND)
- net S2/L3: now also JP1.1 (A); no longer R6.2, U1.B1A (SEL+)
- net S3/R3: now also JP2.1 (A); no longer R7.2, U2.B1A (SEL+)
- net VIN: now also J7.2 (Pin_2)
- new net: C4.2, J7.3 (Pin_3), U3.2 (VO)
- new net: JP2.2 (B), R7.2, U2.B1A (SEL+)
- new net: JP1.2 (B), R6.2, U1.B1A (SEL+)
- new net PLUS: C2.2, J7.1 (Pin_1), J8.2 (Pin_2), U3.3 (VI)

Commit message: PCB fix
Connections:
- net 3V3 is gone; now on net 3.3V: J1.11 (Pin_11), J2.15 (Pin_15), J2.6 (Pin_6), R6.1, R7.1, U1.H1 (H+), U1.V1 (V+), U2.H1 (H+), U2.V1 (V+)
- net G is gone; now on net GND: J1.10 (Pin_10), J1.14 (Pin_14), J1.2 (Pin_2), J2.14 (Pin_14), J2.7 (Pin_7), J8.1 (Pin_1)
- net 3.3V: now also C1.2, C3.2, C5.2, C7.2, D1.1 (VDD), D3.1 (VDD), D5.1 (VDD), D7.1 (VDD)
- net 5V: no longer C1.2, C3.2, C5.2, C7.2, D1.1 (VDD), D3.1 (VDD), D5.1 (VDD), D7.1 (VDD)
Changed lines of the file:
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@@
+    (stroke (width 0) (type default) (color 0 0 0 0))
+  )
+  (wire (pts (xy 73.152 26.67) (xy 73.152 33.274))
     (stroke (width 0) (type default) (color 0 0 0 0))
   )
@@
     (effects (font (size 1.27 1.27)) (justify left bottom))
   )
-  (label "5V" (at 76.2 130.048 0)
-    (effects (font (size 1.27 1.27)) (justify left bottom))
-  )
   (label "D6{slash}DOUT" (at 245.11 141.986 0)
     (effects (font (size 1.27 1.27)) (justify left bottom))
@@
     (effects (font (size 1.27 1.27)) (justify right bottom))
   )
+  (label "3V3" (at 82.804 33.02 0)
+    (effects (font (size 1.27 1.27)) (justify left bottom))
+  )
   (label "VIN" (at 182.372 74.422 180)
     (effects (font (size 1.27 1.27)) (justify right bottom))
   )
+  (label "3V3" (at 50.546 130.048 0)
+    (effects (font (size 1.27 1.27)) (justify left bottom))
+  )
   (label "D7{slash}DIN" (at 245.11 113.284 0)
     (effects (font (size 1.27 1.27)) (justify left bottom))
@@
     (effects (font (size 1.27 1.27)) (justify left bottom))
   )
+  (label "G" (at 73.152 26.67 0)
+    (effects (font (size 1.27 1.27)) (justify left bottom))
+  )
   (label "PLUS" (at 92.456 65.024 180)
     (effects (font (size 1.27 1.27)) (justify right bottom))
@@
     (effects (font (size 1.27 1.27)) (justify left bottom))
   )
+  (label "3V3" (at 25.146 130.048 0)
+    (effects (font (size 1.27 1.27)) (justify left bottom))
+  )
   (label "SO" (at 182.372 56.642 180)
     (effects (font (size 1.27 1.27)) (justify right bottom))
@@
     (effects (font (size 1.27 1.27)) (justify right bottom))
   )
+  (label "3V3" (at 101.6 130.048 0)
+    (effects (font (size 1.27 1.27)) (justify left bottom))
+  )
   (label "D1{slash}ATTACK" (at 203.2 41.402 0)
     (effects (font (size 1.27 1.27)) (justify left bottom))
@@
     (effects (font (size 1.27 1.27)) (justify left bottom))
   )
-  (label "5V" (at 101.6 130.048 0)
-    (effects (font (size 1.27 1.27)) (justify left bottom))
-  )
   (label "RIGHTH" (at 167.386 99.822 180)
     (effects (font (size 1.27 1.27)) (justify right bottom))
@@
     (effects (font (size 1.27 1.27)) (justify right bottom))
   )
+  (label "3V3" (at 76.2 130.048 0)
+    (effects (font (size 1.27 1.27)) (justify left bottom))
+  )
   (label "D3" (at 203.2 46.482 0)
     (effects (font (size 1.27 1.27)) (justify left bottom))
@@
     (effects (font (size 1.27 1.27)) (justify left bottom))
   )
-  (label "5V" (at 25.146 130.048 0)
-    (effects (font (size 1.27 1.27)) (justify left bottom))
-  )
   (label "VV" (at 182.372 43.942 180)
     (effects (font (size 1.27 1.27)) (justify right bottom))
@@
   (label "3.3V" (at 68.326 93.98 180)
     (effects (font (size 1.27 1.27)) (justify right bottom))
-  )
-  (label "5V" (at 50.546 130.048 0)
-    (effects (font (size 1.27 1.27)) (justify left bottom))
   )
   (symbol (lib_id "Connector:Conn_01x15_Female") (at 187.452 56.642 0) (unit 1)
@@
     (pin "2")
   )
+  (symbol (lib_id "power:GND") (at 73.152 33.274 0) (unit 1)
+    (in_bom yes) (on_board yes)
+    (property "Reference" "#PWR0102" (id 0) (at 73.152 39.624 0)
+      (effects (font (size 1.27 1.27)) hide)
+    )
+    (property "Value" "GND" (id 1) (at 73.152 37.592 0))
+    (property "Footprint" "" (id 2) (at 73.152 33.274 0)
+      (effects (font (size 1.27 1.27)) hide)
+    )
+    (property "Datasheet" "" (id 3) (at 73.152 33.274 0)
+      (effects (font (size 1.27 1.27)) hide)
+    )
+    (pin "1")
+  )
   (symbol (lib_id "power:GND") (at 37.338 155.194 0) (unit 1)
     (in_bom yes) (on_board yes) (fields_autoplaced)
@@
       (reference "#PWR0101") (unit 1) (value "GND") (footprint "")
     )
+    (path "/cf5e824f-c15b-4c19-aa9c-bb9acc0a0116"
+      (reference "#PWR0102") (unit 1) (value "GND") (footprint "")
+    )
     (path "/43ece291-02dd-4374-913e-07ed0acd3281"
